File: Design/H3BR7.brd (EAGLE design)
At the start: 60 x 34.6 mm, 62 parts, among them P2 HEXABIT_X2_P1_P5, Q10 MMBT3904LT1, Q11 MMBT3904LT1, Q12 MMBT3904LT1, Q13 MMBT3904LT1, Q14 MMBT3904LT1, Q7 MMBT3904LT1, Q8 MMBT3904LT1, Q9 MMBT3904LT1, U1 STM32G0B1CEU6N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

Commit message: -Add Tvs diode -Update the LOGO -Fix the clearance and soldermask  layer issues
Parts:
- added D2: BOURNS_CDSOD323-T03SCBOURNS_CDSOD323-T03SC_0_0, HEXABITZ_RCLS:BOURNS_CDSOD323-T03SC_0
- added TRIMBLE-LOGO1: HEXA-LOGO, HEXABITZ_USER_INTERFACE_PARTS:HEXA-LOGO
Connections:
- net GND: now also D2.1
- net VDD: now also D2.2
Routing:
- net VDD: track 6.10 -> 7.75 mm
- net GND: track 3.01 -> 4.66 mm
- net USART1_TX: track 14.2 -> 14.9 mm
Other:
- board text added: "P4*"
- board text removed: "P4"
